File: MagnetDriver.kicad_pcb (KiCad board)
At the start: 2 copper layers, 100 x 100 mm, 59 parts, among them J1 MAGNET1, J2 MAGNET2, J3 INPUT_JACK, J4 PWR_IN, Q1 2N3904, Q2 TIP122, Q3 TIP32A, Q4 2N3904, Q5 TIP122, Q6 TIP32A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

Commit message: placed components
Parts:
- moved R17 136.3 mm to (87.0, 88.5), turned to 0 degrees
- moved D4 130.6 mm to (84.0, 89.0), turned to 270 degrees
- moved R16 125.6 mm to (87.0, 85.5), turned to 0 degrees
- moved C5 119.5 mm to (82.5, 82.0), turned to 90 degrees
- moved C4 111.1 mm to (58.5, 85.0), turned to 270 degrees
- moved R14 110.7 mm to (87.0, 79.5), turned to 0 degrees
- moved Q4 108.6 mm to (76.5, 79.5), turned to 270 degrees
- moved R15 108.3 mm to (87.0, 82.5)
- moved R11 107.4 mm to (73.0, 85.5)
- moved R10 106.6 mm to (59.5, 104.5), turned to 180 degrees
- moved R13 103.2 mm to (75.2, 85.5), turned to 0 degrees
- moved R12 99.4 mm to (73.0, 82.5), turned to 180 degrees
- moved R1 77.6 mm to (59.5, 107.0), turned to 180 degrees
- moved C1 56.7 mm to (54.5, 85.0), turned to 270 degrees
- moved R8 52.3 mm to (80.5, 61.5), turned to 270 degrees
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Connections:
- R12 pad 1: VDC -> Net-(Q4-Pad2)
- R12 pad 2: Net-(Q4-Pad2) -> VDC
- R3 pad 1: VDC -> Net-(Q1-Pad2)
- R3 pad 2: Net-(Q1-Pad2) -> VDC
Other:
- board text added: "<VDD IN"
- board text added: "SIG IN>"

Commit message: silkscreen stuff
Parts:
- added G***: LOGO, HammerheadAudio:HotSymbol, F.Cu at (146.5, 114.0)
- added G***: LOGO, HammerheadAudio:HotSymbol, F.Cu at (146.5, 86.0)
- added HH_LOGO_15x7.5mm: , HammerheadAudio:HH_LOGO_15x7.5mm, F.Cu at (173.0, 136.0)
- added HH_LOGO_17.5x8.75mm: , HammerheadAudio:HH_LOGO_17.5x8.75mm, F.Cu at (82.5, 118.5)
- added HH_LOGO_25.6x12.8: , HammerheadAudio:HH_LOGO_25.6x12.8, F.Cu at (170.0, 151.0)
- added HH_LOGO_32x16: , HammerheadAudio:HH_LOGO_32x16, B.Cu at (187.0, 128.0)
- moved C2 2.50 mm to (85.0, 73.5)
- moved C5 2.50 mm to (85.0, 82.0)
- moved R1 2.06 mm to (61.5, 106.5)
- moved R10 2.06 mm to (61.5, 104.0)
- moved D4 1.00 mm to (85.0, 89.0)
- moved D5 1.00 mm to (133.5, 131.0)
- moved Q1 1.00 mm to (77.5, 73.5)
- moved Q4 1.00 mm to (77.5, 79.5)
- moved R14 1.00 mm to (88.0, 79.5)
- moved R15 1.00 mm to (88.0, 82.5)
- moved R16 1.00 mm to (88.0, 85.5)
- moved R17 1.00 mm to (88.0, 88.5)
- moved R18 1.00 mm to (130.0, 131.0)
- moved R5 1.00 mm to (88.0, 76.5)
- moved R6 1.00 mm to (88.0, 73.5)
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Connections:
- RV3 pad 1: Net-(C6-Pad2) -> Net-(C6-Pad1)
- RV3 pad 2: Net-(C6-Pad2) -> Net-(C6-Pad1)
- RV3 pad 3: Net-(C6-Pad1) -> Net-(C6-Pad2)
Routing:
- added copper zone on F.Cu, net GND
Other:
- board text added: "! WARNING ! ! HEATSINKS MAY BE HOT !"
- board text added: "M1_GAIN"
- board text added: "M1_IND"
- board text added: "M1_OUT ▶"
- board text added: "M1_VOLUME"
- board text added: "M2_GAIN"
- board text added: "M2_IND"
- board text added: "M2_VOLUME"
- board text added: "PWR_IND"
- board text added: "STEREO MAGNET DRIVER V0.1 HAMMERHEAD AUDIO X ERIC HEEP DESIGN BY EMMETT PALAIMA JAN. 2021"
- board text added: "◀ M2_OUT"
- board text added: "◀ PWR_IN : 9V-24V"
- board text added: "◀ SIG_IN"
- board text removed: "<VDD IN"
- board text removed: "SIG IN>"

Commit message: finished first layout
Parts:
- removed HH_LOGO_15x7.5mm: , HammerheadAudio:HH_LOGO_15x7.5mm
- removed HH_LOGO_25.6x12.8: , HammerheadAudio:HH_LOGO_25.6x12.8
- removed HH_LOGO_32x16: , HammerheadAudio:HH_LOGO_32x16
- moved D1 1.58 mm to (85.0, 69.8)
- moved R7 1.00 mm to (78.5, 61.5)
- moved R8 1.00 mm to (81.5, 61.5)
- moved R10 0.50 mm to (61.5, 103.5)
- moved C7 0.25 mm to (74.0, 64.2)
Routing:
- net VDC: track 0.00 -> 427.4 mm
- net Net-(C6-Pad2): track 0.00 -> 82.5 mm
- net Net-(C3-Pad1): track 0.00 -> 75.0 mm
- net Net-(C3-Pad2): track 0.00 -> 74.2 mm
- net Net-(RV2-Pad3): track 0.00 -> 56.2 mm
- net Net-(C6-Pad1): track 0.00 -> 49.6 mm
- net Net-(RV4-Pad3): track 0.00 -> 48.2 mm
- net Net-(D5-Pad1): track 0.00 -> 44.9 mm
- net Net-(D2-Pad1): track 0.00 -> 43.3 mm
- net Net-(Q5-Pad1): track 0.00 -> 41.8 mm
- net Net-(Q2-Pad1): track 0.00 -> 39.7 mm
- net +5V: track 0.00 -> 36.0 mm
- net IN_L: track 0.00 -> 23.7 mm
- net TEENSY_R: track 0.00 -> 23.2 mm
- net IN_R: track 0.00 -> 17.2 mm
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- added copper zone on F.Cu, net (none)
Other:
- board text added: "M1=T/L"
- board text added: "M1_OUT(T/L) ▶"
- board text added: "◀ M2_OUT(R/R)"
- board text removed: "M1_OUT ▶"
- board text removed: "◀ M2_OUT"
