File: MagnetDriver.kicad_pcb (KiCad board)
At the start: 2 copper layers, 100 x 100 mm, 62 parts, among them J1 MAGNET1, J2 MAGNET2, J3 INPUT_JACK, J4 PWR_IN, Q1 2N3904, Q2 TIP122, Q3 TIP32A, Q4 2N3904, Q5 TIP122, Q6 TIP32A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

Commit message: testing adding teesny switch
Other:
- board text removed: "M1=T/L"
Changed lines of the file:
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@@
   (general
     (thickness 1.6)
-    (drawings 22)
-    (tracks 264)
+    (drawings 23)
+    (tracks 265)
     (zones 0)
     (modules 62)
@@
   )
   (setup
-    (last_trace_width 0.25)
+    (last_trace_width 2.5)
     (user_trace_width 0.5)
     (user_trace_width 1)
@@
       (net 20 "Net-(D5-Pad1)"))
     (pad "" np_thru_hole circle (at 12.7 0 180) (size 3.3 3.3) (drill 2.7) (layers *.Cu *.Mask)
-      (clearance 1))
+      (clearance 2))
     (pad "" np_thru_hole circle (at -12.7 0 180) (size 3.3 3.3) (drill 2.7) (layers *.Cu *.Mask)
-      (clearance 1))
+      (clearance 2))
   )
   (module HammerheadAudio:TO-220_BigHeatsink (layer F.Cu)
@@
       (net 17 "Net-(D2-Pad1)"))
     (pad "" np_thru_hole circle (at 12.7 0) (size 3.3 3.3) (drill 2.7) (layers *.Cu *.Mask)
-      (clearance 1))
+      (clearance 2))
     (pad "" np_thru_hole circle (at -12.7 0) (size 3.3 3.3) (drill 2.7) (layers *.Cu *.Mask)
-      (clearance 1))
+      (clearance 2))
   )
   (module HammerheadAudio:HH_LOGO_17.5x8.75mm (layer F.Cu)
@@
     )
   )
+  (dimension 16 (width 0.15) (layer Cmts.User)
+    (gr_text "16.000 mm" (at 34.7 132 270) (layer Cmts.User)
+      (effects (font (size 1 1) (thickness 0.15)))
+    )
+    (feature1 (pts (xy 56.75 140) (xy 35.413579 140)))
+    (feature2 (pts (xy 56.75 124) (xy 35.413579 124)))
+    (crossbar (pts (xy 36 124) (xy 36 140)))
+    (arrow1a (pts (xy 36 140) (xy 35.413579 138.873496)))
+    (arrow1b (pts (xy 36 140) (xy 36.586421 138.873496)))
+    (arrow2a (pts (xy 36 124) (xy 35.413579 125.126504)))
+    (arrow2b (pts (xy 36 124) (xy 36.586421 125.126504)))
+  )
+  (dimension 16 (width 0.15) (layer Cmts.User)
+    (gr_text "16.000 mm" (at 34.7 116 90) (layer Cmts.User)
+      (effects (font (size 1 1) (thickness 0.15)))
+    )
+    (feature1 (pts (xy 56.75 108) (xy 35.413579 108)))
+    (feature2 (pts (xy 56.75 124) (xy 35.413579 124)))
+    (crossbar (pts (xy 36 124) (xy 36 108)))
+    (arrow1a (pts (xy 36 108) (xy 36.586421 109.126504)))
+    (arrow1b (pts (xy 36 108) (xy 35.413579 109.126504)))
+    (arrow2a (pts (xy 36 124) (xy 36.586421 122.873496)))
+    (arrow2b (pts (xy 36 124) (xy 35.413579 122.873496)))
+  )
   (dimension 100 (width 0.15) (layer Cmts.User)
     (gr_text "100.000 mm" (at 100 38.7) (layer Cmts.User)
@@
     (arrow2b (pts (xy 45 55) (xy 45.586421 56.126504)))
   )
-  (gr_text M1=T/L (at 96.25 148.5) (layer F.SilkS)
-    (effects (font (size 1 1) (thickness 0.15)))
-  )
   (gr_text PWR_IND (at 68 55 270) (layer F.SilkS)
     (effects (font (size 1 1) (thickness 0.15)))
@@
   (segment (start 119.46 110.25) (end 119.46 115.71) (width 2.5) (layer F.Cu) (net 20))
   (segment (start 119.46 115.71) (end 119.46 117.96) (width 2.5) (layer F.Cu) (net 20))
-  (segment (start 128.5 129.5) (end 130 131) (width 2.5) (layer F.Cu) (net 20))
-  (segment (start 128.5 117.437498) (end 128.5 129.5) (width 2.5) (layer F.Cu) (net 20))
+  (segment (start 130 130) (end 130 131) (width 2.5) (layer F.Cu) (net 20))
+  (segment (start 128.5 128.5) (end 130 130) (width 2.5) (layer F.Cu) (net 20))
+  (segment (start 128.5 117.437498) (end 128.5 128.5) (width 2.5) (layer F.Cu) (net 20))
   (segment (start 126.612492 115.54999) (end 128.5 117.437498) (width 2.5) (layer F.Cu) (net 20))
   (segment (start 136.4 141.8) (end 137.54 142.94) (width 0.25) (layer F.Cu) (net 21))

Commit message: backup before layout changes
Parts:
- added D9: LED, LED_THT:LED_D5.0mm, F.Cu at (56.5, 135.5)
- added HH_LOGO_32x16: , HammerheadAudio:HH_LOGO_32x16, B.Cu at (138.0, 92.0)
- added Q7: 2N3904, Package_TO_SOT_THT:TO-92_Inline, F.Cu at (73.5, 119.8)
- added R20: 220, HammerheadAudio:R_THT_P7.62, F.Cu at (61.5, 109.8)
- added R21: 1k, HammerheadAudio:R_THT_P7.62, F.Cu at (61.5, 112.8)
- added R22: 100k, HammerheadAudio:R_THT_P7.62, F.Cu at (76.0, 115.5)
- added SW1: SW_SPDT, HammerheadAudio:Tayda_Slide_SPDT, F.Cu at (56.5, 124.0)
- U3: value LM7805_TO220 -> R-78E5.0-0.5; footprint Package_TO_SOT_THT:TO-220-3_Horizontal_TabDown -> Converter_DCDC:Converter_DCDC_RECOM_R-78E-0.5_THT
- moved C8 12.0 mm to (69.8, 131.0)
- moved C9 12.0 mm to (74.8, 131.0)
- moved U3 12.0 mm to (74.8, 134.5)
- moved HH_LOGO_17.5x8.75mm 1.50 mm to (82.5, 117.0)
- moved D3 0.50 mm to (135.5, 55.0)
- moved D6 0.50 mm to (135.5, 145.0)
- moved D8 0.50 mm to (64.5, 55.0)
Connections:
- RV3 pad 1: Net-(C6-Pad1) -> Net-(C6-Pad2)
- RV3 pad 2: Net-(C6-Pad1) -> Net-(C6-Pad2)
- RV3 pad 3: Net-(C6-Pad2) -> Net-(C6-Pad1)
- U2 pad 48: +5V -> Net-(SW1-Pad3)
Routing:
- net Net-(R20-Pad2): track 0.00 -> 41.1 mm
- net Net-(Q7-Pad3): track 0.00 -> 37.8 mm
- net Net-(D9-Pad2): track 0.00 -> 37.1 mm
- net Net-(SW1-Pad3): track 0.00 -> 31.1 mm
- net VDC: track 427.4 -> 405.0 mm
- net +5V: track 36.0 -> 20.8 mm
- net Net-(Q7-Pad2): track 0.00 -> 14.5 mm
- net Net-(R21-Pad2): track 0.00 -> 9.34 mm
- net Net-(C6-Pad2): track 82.5 -> 75.5 mm
- net Net-(C6-Pad1): track 49.6 -> 47.2 mm
- net Net-(D8-Pad2): track 12.3 -> 13.3 mm
- net Net-(D6-Pad2): track 12.1 -> 12.6 mm
Other:
- board text added: "MICRO_IND"
- board text added: "OFF<-MICRO->ON"
